Commit message: add Robowflex

File: single_arm_v12_plus/urdf/single_arm_v12_plus.urdf (robot description, URDF)
Before this commit: robot single_arm_v12, 8 links, 7 joints
Links:
- link Link1: mass 0.38613 -> 0.386131223153925; geometry collision mesh filename=package://single_arm_v12_plus/meshes/Link1.STL; visual mesh filename=package://single_arm_v12_plus/meshes/Link1.STL
- link Link2: mass 0.61539 -> 0.615390607724248; geometry collision mesh filename=package://single_arm_v12_plus/meshes/Link2.STL; visual mesh filename=package://single_arm_v12_plus/meshes/Link2.STL
- link Link3: geometry collision mesh filename=package://single_arm_v12_plus/meshes/Link3.STL; visual mesh filename=package://single_arm_v12_plus/meshes/Link3.STL
- link Link4: mass 0.313854171959486 -> 0.31385; geometry collision mesh filename=package://single_arm_v12_plus/meshes/Link4.STL; visual mesh filename=package://single_arm_v12_plus/meshes/Link4.STL
- link Link5: mass 0.313854171959487 -> 0.31385; geometry collision mesh filename=package://single_arm_v12_plus/meshes/Link5.STL; visual mesh filename=package://single_arm_v12_plus/meshes/Link5.STL
- link Link6: geometry collision mesh filename=package://single_arm_v12_plus/meshes/Link6.STL; visual mesh filename=package://single_arm_v12_plus/meshes/Link6.STL
- link base_link: mass 0.47711 -> 0.477111748769872; geometry collision mesh filename=package://single_arm_v12_plus/meshes/base_link.STL; visual mesh filename=package://single_arm_v12_plus/meshes/base_link.STL
Joints:
- joint Joint2: origin xyz=0 -0.0685 0.0315 rpy=1.5708 0 0 -> xyz=0 -0.0685 0.0315 rpy=1.5707963267949 0 0
- joint Joint4: origin xyz=0.214 0 0.0325 rpy=0 0 3.1416 -> xyz=0.214 0 0.0325 rpy=0 0 -3.1416
- joint Joint6: origin xyz=0.0346 0.068329 -0.0048371 rpy=1.5708 -1.5708 0 -> xyz=0.0346 0.0685 0 rpy=1.5708 -1.5708 0
